Commit message: Add new meshes to URDF file

File: src/rover_description/urdf/robot.urdf (robot description, URDF)
Before this commit: robot scarab, 10 links, 9 joints
Links:
- link body_link: geometry collision mesh filename=package://rover_description/meshes/base_link.stl scale=0.001 0.001 0.001; visual mesh filename=package://rover_description/meshes/base_link.stl scale=0.001 0.001 0.001
- link susLeft_link: geometry collision mesh filename=package://rover_description/meshes/suspension_left_link.stl scale=0.001 0.001 0.001; visual mesh filename=package://rover_description/meshes/suspension_left_link.stl scale=0.001 0.001 0.001
- link susRight_link: geometry collision mesh filename=package://rover_description/meshes/suspension_right_link.stl scale=0.001 0.001 0.001; visual mesh filename=package://rover_description/meshes/suspension_right_link.stl scale=0.001 0.001 0.001
