Commit message: Simulate suspension on right side

File: src/rover_description/urdf/rover.urdf.xacro (robot description, xacro)
@@ -22,5 +22,5 @@
         </inertial>
         <visual>
-            <origin rpy="0 0 1.579795" xyz="0 0.03 0"/>
+            <origin rpy="0 0 1.579795" xyz="0 0 0"/>
             <geometry>
                 <!--<box size="1 0.6 0.3"/>-->
@@ -32,5 +32,5 @@
         </visual>
         <collision>
-            <origin rpy="0 0 1.579795" xyz="0 0.03 0"/>
+            <origin rpy="0 0 1.579795" xyz="0 0 0"/>
             <geometry>
                 <mesh filename="package://rover_description/meshes/base_link.stl" scale="0.001 0.001 0.001" />
@@ -42,5 +42,5 @@
         <parent link="body_link" />
         <child link="susLeft_link" />
-        <origin xyz ="-0.1 -0.17 0.04" rpy="0 0 -1.579795" />
+        <origin xyz ="-0.1 -0.2 0.04" rpy="0 0 -1.579795" />
         <axis xyz="1 0 0" />
     </joint>
@@ -71,5 +71,5 @@
         <parent link="body_link" />
         <child link="susRight_link" />
-        <origin xyz ="-0.1 0.23 0.04" rpy="0 0 -1.579795" />
+        <origin xyz ="-0.1 0.21 0.04" rpy="0 0 -1.579795" />
         <axis xyz="1 0 0" />
     </joint>
@@ -83,5 +83,5 @@
             <origin rpy="0 0 0" xyz="0 0 0"/>
             <geometry>
-                <mesh filename="package://rover_description/meshes/suspension_right_link.stl" scale="0.001 0.001 0.001" />
+                <mesh filename="package://rover_description/meshes/suspension_right_link_b.stl" scale="0.001 0.001 0.001" />
             </geometry>
             <material name="yellow">
@@ -92,5 +92,33 @@
             <origin rpy="0 0 0" xyz="0 0 0"/>
             <geometry>
-                <mesh filename="package://rover_description/meshes/suspension_right_link.stl" scale="0.001 0.001 0.001" />
+                <mesh filename="package://rover_description/meshes/suspension_right_link_b.stl" scale="0.001 0.001 0.001" />
+            </geometry>
+        </collision>
+    </link>
+    <joint name="susRight_joint_b" type="continuous">
+        <parent link="susRight_link" />
+        <child link="susRight_link_b" />
+        <origin xyz ="-0.038 -0.156485 -0.088953" rpy="0 0 0" />
+        <axis xyz="1 0 0" />
+    </joint>
+    <link name="susRight_link_b">
+        <inertial>
+            <origin xyz="0 0 0" rpy="0 0 0"/>
+            <mass value="2.0"/>
+            <inertia ixx="0.1" ixy="0.0" ixz="0.0" iyy="0.1" iyz="0.0" izz="0.1"/>
+        </inertial>
+        <visual>
+            <origin rpy="0 0 0" xyz="0 0 0"/>
+            <geometry>
+                <mesh filename="package://rover_description/meshes/suspension_right_link_a.stl" scale="0.001 0.001 0.001" />
+            </geometry>
+            <material name="yellow">
+                <color rgba="1 1 0 1"/>
+            </material>
+        </visual>
+        <collision>
+            <origin rpy="0 0 0" xyz="0 0 0"/>
+            <geometry>
+                <mesh filename="package://rover_description/meshes/suspension_right_link_a.stl" scale="0.001 0.001 0.001" />
             </geometry>
         </collision>
@@ -98,7 +126,7 @@
     <!-- This is the front right wheel of the rover -->
     <joint name="wheel1_joint" type="continuous">
-        <parent link="susRight_link" />
+        <parent link="susRight_link_b" />
         <child link="wheel1_link" />
-        <origin xyz ="-0.1 -0.35 -0.3" rpy="0 0 0" />
+        <origin xyz ="-0.05 -0.20796 -0.196506" rpy="0 0 0" />
         <axis xyz="1 0 0" />
     </joint>
@@ -112,14 +140,14 @@
             <origin rpy="1.579795 0 1.579795" xyz="0 0 0"/>
             <geometry>
-                <cylinder radius="0.123" length="0.12"/>
-            </geometry>
-            <material name="black">
-                <color rgba="0.01 0.01 0.01 1"/>
-            </material>
-        </visual>
-        <collision>
-            <origin rpy="1.579795 0 1.579795" xyz="0 0 0"/>
-            <geometry>
-                <cylinder radius="0.123" length="0.12"/>
+                <cylinder radius="0.1175" length="0.12"/>
+            </geometry>
+            <material name="black">
+                <color rgba="0.01 0.01 0.01 1"/>
+            </material>
+        </visual>
+        <collision>
+            <origin rpy="1.579795 0 1.579795" xyz="0 0 0"/>
+            <geometry>
+                <cylinder radius="0.1175" length="0.12"/>
             </geometry>
         </collision>
@@ -141,14 +169,14 @@
             <origin rpy="1.579795 0 1.579795" xyz="0 0 0"/>
             <geometry>
-                <cylinder radius="0.123" length="0.12"/>
-            </geometry>
-            <material name="black">
-                <color rgba="0.01 0.01 0.01 1"/>
-            </material>
-        </visual>
-        <collision>
-            <origin rpy="1.579795 0 1.579795" xyz="0 0 0"/>
-            <geometry>
-                <cylinder radius="0.123" length="0.12"/>
+                <cylinder radius="0.1175" length="0.12"/>
+            </geometry>
+            <material name="black">
+                <color rgba="0.01 0.01 0.01 1"/>
+            </material>
+        </visual>
+        <collision>
+            <origin rpy="1.579795 0 1.579795" xyz="0 0 0"/>
+            <geometry>
+                <cylinder radius="0.1175" length="0.12"/>
             </geometry>
         </collision>
@@ -156,7 +184,7 @@
     <!-- This is the middle right wheel of the rover -->
     <joint name="wheel3_joint" type="continuous">
-        <parent link="susRight_link" />
+        <parent link="susRight_link_b" />
         <child link="wheel3_link" />
-        <origin xyz ="-0.19 0.01 -0.3" rpy="0 0 0" />
+        <origin xyz ="-0.11 0.168268 -0.211155" rpy="0 0 0" />
         <axis xyz="1 0 0" />
     </joint>
@@ -170,14 +198,14 @@
             <origin rpy="1.579795 0 1.579795" xyz="0 0 0"/>
             <geometry>
-                <cylinder radius="0.123" length="0.12"/>
-            </geometry>
-            <material name="black">
-                <color rgba="0.01 0.01 0.01 1"/>
-            </material>
-        </visual>
-        <collision>
-            <origin rpy="1.579795 0 1.579795" xyz="0 0 0"/>
-            <geometry>
-                <cylinder radius="0.123" length="0.12"/>
+                <cylinder radius="0.1175" length="0.12"/>
+            </geometry>
+            <material name="black">
+                <color rgba="0.01 0.01 0.01 1"/>
+            </material>
+        </visual>
+        <collision>
+            <origin rpy="1.579795 0 1.579795" xyz="0 0 0"/>
+            <geometry>
+                <cylinder radius="0.1175" length="0.12"/>
             </geometry>
         </collision>
@@ -199,14 +227,14 @@
             <origin rpy="1.579795 0 1.579795" xyz="0 0 0"/>
             <geometry>
-                <cylinder radius="0.123" length="0.12"/>
-            </geometry>
-            <material name="black">
-                <color rgba="0.01 0.01 0.01 1"/>
-            </material>
-        </visual>
-        <collision>
-            <origin rpy="1.579795 0 1.579795" xyz="0 0 0"/>
-            <geometry>
-                <cylinder radius="0.123" length="0.12"/>
+                <cylinder radius="0.1175" length="0.12"/>
+            </geometry>
+            <material name="black">
+                <color rgba="0.01 0.01 0.01 1"/>
+            </material>
+        </visual>
+        <collision>
+            <origin rpy="1.579795 0 1.579795" xyz="0 0 0"/>
+            <geometry>
+                <cylinder radius="0.1175" length="0.12"/>
             </geometry>
         </collision>
@@ -228,14 +256,14 @@
             <origin rpy="1.579795 0 1.579795" xyz="0 0 0"/>
             <geometry>
-                <cylinder radius="0.123" length="0.12"/>
-            </geometry>
-            <material name="black">
-                <color rgba="0.01 0.01 0.01 1"/>
-            </material>
-        </visual>
-        <collision>
-            <origin rpy="1.579795 0 1.579795" xyz="0 0 0"/>
-            <geometry>
-                <cylinder radius="0.123" length="0.12"/>
+                <cylinder radius="0.1175" length="0.12"/>
+            </geometry>
+            <material name="black">
+                <color rgba="0.01 0.01 0.01 1"/>
+            </material>
+        </visual>
+        <collision>
+            <origin rpy="1.579795 0 1.579795" xyz="0 0 0"/>
+            <geometry>
+                <cylinder radius="0.1175" length="0.12"/>
             </geometry>
         </collision>
@@ -257,14 +285,14 @@
             <origin rpy="1.579795 0 1.579795" xyz="0 0 0"/>
             <geometry>
-                <cylinder radius="0.123" length="0.12"/>
-            </geometry>
-            <material name="black">
-                <color rgba="0.01 0.01 0.01 1"/>
-            </material>
-        </visual>
-        <collision>
-            <origin rpy="1.579795 0 1.579795" xyz="0 0 0"/>
-            <geometry>
-                <cylinder radius="0.123" length="0.12"/>
+                <cylinder radius="0.1175" length="0.12"/>
+            </geometry>
+            <material name="black">
+                <color rgba="0.01 0.01 0.01 1"/>
+            </material>
+        </visual>
+        <collision>
+            <origin rpy="1.579795 0 1.579795" xyz="0 0 0"/>
+            <geometry>
+                <cylinder radius="0.1175" length="0.12"/>
             </geometry>
         </collision>

Commit message: Add suspension to left side

File: src/rover_description/urdf/rover.urdf.xacro (robot description, xacro)
@@ -42,5 +42,5 @@
         <parent link="body_link" />
         <child link="susLeft_link" />
-        <origin xyz ="-0.1 -0.2 0.04" rpy="0 0 -1.579795" />
+        <origin xyz ="-0.1 -0.239 0.04" rpy="0 0 -1.579795" />
         <axis xyz="1 0 0" />
     </joint>
@@ -54,14 +54,14 @@
             <origin rpy="0 0 0" xyz="0 0 0"/>
             <geometry>
-                <mesh filename="package://rover_description/meshes/suspension_left_link.stl" scale="0.001 0.001 0.001" />
-            </geometry>
-            <material name="yellow">
-                <color rgba="1 1 0 1"/>
-            </material>
-        </visual>
-        <collision>
-            <origin rpy="0 0 0" xyz="0 0 0"/>
-            <geometry>
-                <mesh filename="package://rover_description/meshes/suspension_left_link.stl" scale="0.001 0.001 0.001" />
+                <mesh filename="package://rover_description/meshes/suspension_left_link_b.stl" scale="0.001 0.001 0.001" />
+            </geometry>
+            <material name="yellow">
+                <color rgba="1 1 0 1"/>
+            </material>
+        </visual>
+        <collision>
+            <origin rpy="0 0 0" xyz="0 0 0"/>
+            <geometry>
+                <mesh filename="package://rover_description/meshes/suspension_left_link_b.stl" scale="0.001 0.001 0.001" />
             </geometry>
         </collision>
@@ -124,4 +124,32 @@
         </collision>
     </link>
+    <joint name="susLeft_joint_b" type="continuous">
+        <parent link="susLeft_link" />
+        <child link="susLeft_link_b" />
+        <origin xyz ="0.052 -0.156485 -0.088953" rpy="0 0 0" />
+        <axis xyz="1 0 0" />
+    </joint>
+    <link name="susLeft_link_b">
+        <inertial>
+            <origin xyz="0 0 0" rpy="0 0 0"/>
+            <mass value="2.0"/>
+            <inertia ixx="0.1" ixy="0.0" ixz="0.0" iyy="0.1" iyz="0.0" izz="0.1"/>
+        </inertial>
+        <visual>
+            <origin rpy="0 0 0" xyz="0 0 0"/>
+            <geometry>
+                <mesh filename="package://rover_description/meshes/suspension_left_link_a.stl" scale="0.001 0.001 0.001" />
+            </geometry>
+            <material name="yellow">
+                <color rgba="1 1 0 1"/>
+            </material>
+        </visual>
+        <collision>
+            <origin rpy="0 0 0" xyz="0 0 0"/>
+            <geometry>
+                <mesh filename="package://rover_description/meshes/suspension_left_link_a.stl" scale="0.001 0.001 0.001" />
+            </geometry>
+        </collision>
+    </link>
     <!-- This is the front right wheel of the rover -->
     <joint name="wheel1_joint" type="continuous">
@@ -155,7 +183,7 @@
     <!-- This is the front left wheel of the rover -->
     <joint name="wheel2_joint" type="continuous">
-        <parent link="susLeft_link" />
+        <parent link="susLeft_link_b" />
         <child link="wheel2_link" />
-        <origin xyz ="0.1 -0.35 -0.3" rpy="0 0 0" />
+        <origin xyz ="0.05 -0.20796 -0.196506" rpy="0 0 0" />
         <axis xyz="1 0 0" />
     </joint>
@@ -213,7 +241,7 @@
     <!-- This is the middle left wheel of the rover -->
     <joint name="wheel4_joint" type="continuous">
-        <parent link="susLeft_link" />
+        <parent link="susLeft_link_b" />
         <child link="wheel4_link" />
-        <origin xyz ="0.19 0.01 -0.3" rpy="0 0 0" />
+        <origin xyz ="0.1 0.168268 -0.211155" rpy="0 0 0" />
         <axis xyz="1 0 0" />
     </joint>
@@ -273,5 +301,5 @@
         <parent link="susLeft_link" />
         <child link="wheel6_link" />
-        <origin xyz ="0.05 0.35 -0.3" rpy="0 0 0" />
+        <origin xyz ="0.02 0.35 -0.3" rpy="0 0 0" />
         <axis xyz="1 0 0" />
     </joint>

Commit message: Fix joint transforms in gazebo control

File: src/rover_description/urdf/rover.urdf.xacro (robot description, xacro)
@@ -54,14 +54,14 @@
             <origin rpy="0 0 0" xyz="0 0 0"/>
             <geometry>
-                <mesh filename="package://rover_description/meshes/suspension_left_link_b.stl" scale="0.001 0.001 0.001" />
-            </geometry>
-            <material name="yellow">
-                <color rgba="1 1 0 1"/>
-            </material>
-        </visual>
-        <collision>
-            <origin rpy="0 0 0" xyz="0 0 0"/>
-            <geometry>
-                <mesh filename="package://rover_description/meshes/suspension_left_link_b.stl" scale="0.001 0.001 0.001" />
+                <mesh filename="package://rover_description/meshes/suspension_left_link_a.stl" scale="0.001 0.001 0.001" />
+            </geometry>
+            <material name="yellow">
+                <color rgba="1 1 0 1"/>
+            </material>
+        </visual>
+        <collision>
+            <origin rpy="0 0 0" xyz="0 0 0"/>
+            <geometry>
+                <mesh filename="package://rover_description/meshes/suspension_left_link_a.stl" scale="0.001 0.001 0.001" />
             </geometry>
         </collision>
@@ -83,14 +83,14 @@
             <origin rpy="0 0 0" xyz="0 0 0"/>
             <geometry>
-                <mesh filename="package://rover_description/meshes/suspension_right_link_b.stl" scale="0.001 0.001 0.001" />
-            </geometry>
-            <material name="yellow">
-                <color rgba="1 1 0 1"/>
-            </material>
-        </visual>
-        <collision>
-            <origin rpy="0 0 0" xyz="0 0 0"/>
-            <geometry>
-                <mesh filename="package://rover_description/meshes/suspension_right_link_b.stl" scale="0.001 0.001 0.001" />
+                <mesh filename="package://rover_description/meshes/suspension_right_link_a.stl" scale="0.001 0.001 0.001" />
+            </geometry>
+            <material name="yellow">
+                <color rgba="1 1 0 1"/>
+            </material>
+        </visual>
+        <collision>
+            <origin rpy="0 0 0" xyz="0 0 0"/>
+            <geometry>
+                <mesh filename="package://rover_description/meshes/suspension_right_link_a.stl" scale="0.001 0.001 0.001" />
             </geometry>
         </collision>
@@ -111,14 +111,14 @@
             <origin rpy="0 0 0" xyz="0 0 0"/>
             <geometry>
-                <mesh filename="package://rover_description/meshes/suspension_right_link_a.stl" scale="0.001 0.001 0.001" />
-            </geometry>
-            <material name="yellow">
-                <color rgba="1 1 0 1"/>
-            </material>
-        </visual>
-        <collision>
-            <origin rpy="0 0 0" xyz="0 0 0"/>
-            <geometry>
-                <mesh filename="package://rover_description/meshes/suspension_right_link_a.stl" scale="0.001 0.001 0.001" />
+                <mesh filename="package://rover_description/meshes/suspension_right_link_b.stl" scale="0.001 0.001 0.001" />
+            </geometry>
+            <material name="yellow">
+                <color rgba="1 1 0 1"/>
+            </material>
+        </visual>
+        <collision>
+            <origin rpy="0 0 0" xyz="0 0 0"/>
+            <geometry>
+                <mesh filename="package://rover_description/meshes/suspension_right_link_b.stl" scale="0.001 0.001 0.001" />
             </geometry>
         </collision>
@@ -139,14 +139,14 @@
             <origin rpy="0 0 0" xyz="0 0 0"/>
             <geometry>
-                <mesh filename="package://rover_description/meshes/suspension_left_link_a.stl" scale="0.001 0.001 0.001" />
-            </geometry>
-            <material name="yellow">
-                <color rgba="1 1 0 1"/>
-            </material>
-        </visual>
-        <collision>
-            <origin rpy="0 0 0" xyz="0 0 0"/>
-            <geometry>
-                <mesh filename="package://rover_description/meshes/suspension_left_link_a.stl" scale="0.001 0.001 0.001" />
+                <mesh filename="package://rover_description/meshes/suspension_left_link_b.stl" scale="0.001 0.001 0.001" />
+            </geometry>
+            <material name="yellow">
+                <color rgba="1 1 0 1"/>
+            </material>
+        </visual>
+        <collision>
+            <origin rpy="0 0 0" xyz="0 0 0"/>
+            <geometry>
+                <mesh filename="package://rover_description/meshes/suspension_left_link_b.stl" scale="0.001 0.001 0.001" />
             </geometry>
         </collision>

File: src/rover_description/urdf/rover_control.xacro (robot description, xacro)
@@ -14,4 +14,20 @@
             </hardware>
         </xacro:unless>
+        <joint name="susLeft_joint_b">
+            <command_interface name="velocity">
+                <param name="min">-1</param>
+                <param name="max">1</param>
+            </command_interface>
+            <state_interface name="position" />
+            <state_interface name="velocity" />
+        </joint>
+        <joint name="susRight_joint_b">
+            <command_interface name="velocity">
+                <param name="min">-1</param>
+                <param name="max">1</param>
+            </command_interface>
+            <state_interface name="position" />
+            <state_interface name="velocity" />
+        </joint>
         <joint name="wheel1_joint">
             <command_interface name="velocity">
