Commit message: Fix: gazebo sus_joint control does not move because velocity was published

File: src/rover_description/urdf/rover.urdf.xacro (robot description, xacro)
@@ -67,4 +67,34 @@
         </collision>
     </link>
+    <joint name="susLeft_joint_b" type="continuous">
+        <parent link="susLeft_link" />
+        <child link="susLeft_link_b" />
+        <origin xyz ="0.052 -0.156485 -0.088953" rpy="0 0 0" />
+        <axis xyz="1 0 0" />
+        <dynamics damping="0.1" friction="0.1"/>
+        <limit effort="50" velocity="1"/>
+    </joint>
+    <link name="susLeft_link_b">
+        <inertial>
+            <origin xyz="0 0 0" rpy="0 0 0"/>
+            <mass value="2.0"/>
+            <inertia ixx="0.1" ixy="0.0" ixz="0.0" iyy="0.1" iyz="0.0" izz="0.1"/>
+        </inertial>
+        <visual>
+            <origin rpy="0 0 0" xyz="0 0 0"/>
+            <geometry>
+                <mesh filename="package://rover_description/meshes/suspension_left_link_b.stl" scale="0.001 0.001 0.001" />
+            </geometry>
+            <material name="yellow">
+                <color rgba="1 1 0 1"/>
+            </material>
+        </visual>
+        <collision>
+            <origin rpy="0 0 0" xyz="0 0 0"/>
+            <geometry>
+                <mesh filename="package://rover_description/meshes/suspension_left_link_b.stl" scale="0.001 0.001 0.001" />
+            </geometry>
+        </collision>
+    </link>
     <!-- This is the right suspension assembly -->
     <joint name="susRight_joint" type="fixed">
@@ -73,4 +103,6 @@
         <origin xyz ="-0.1 0.21 0.04" rpy="0 0 -1.579795" />
         <axis xyz="1 0 0" />
+        <dynamics damping="0.1" friction="0.1"/>
+        <limit effort="50" velocity="1"/>
     </joint>
     <link name="susRight_link">
@@ -121,32 +153,4 @@
             <geometry>
                 <mesh filename="package://rover_description/meshes/suspension_right_link_b.stl" scale="0.001 0.001 0.001" />
-            </geometry>
-        </collision>
-    </link>
-    <joint name="susLeft_joint_b" type="continuous">
-        <parent link="susLeft_link" />
-        <child link="susLeft_link_b" />
-        <origin xyz ="0.052 -0.156485 -0.088953" rpy="0 0 0" />
-        <axis xyz="1 0 0" />
-    </joint>
-    <link name="susLeft_link_b">
-        <inertial>
-            <origin xyz="0 0 0" rpy="0 0 0"/>
-            <mass value="2.0"/>
-            <inertia ixx="0.1" ixy="0.0" ixz="0.0" iyy="0.1" iyz="0.0" izz="0.1"/>
-        </inertial>
-        <visual>
-            <origin rpy="0 0 0" xyz="0 0 0"/>
-            <geometry>
-                <mesh filename="package://rover_description/meshes/suspension_left_link_b.stl" scale="0.001 0.001 0.001" />
-            </geometry>
-            <material name="yellow">
-                <color rgba="1 1 0 1"/>
-            </material>
-        </visual>
-        <collision>
-            <origin rpy="0 0 0" xyz="0 0 0"/>
-            <geometry>
-                <mesh filename="package://rover_description/meshes/suspension_left_link_b.stl" scale="0.001 0.001 0.001" />
             </geometry>
         </collision>

File: src/rover_description/urdf/rover_control.xacro (robot description, xacro)
@@ -15,18 +15,8 @@
         </xacro:unless>
         <joint name="susLeft_joint_b">
-            <command_interface name="velocity">
-                <param name="min">-1</param>
-                <param name="max">1</param>
-            </command_interface>
             <state_interface name="position" />
-            <state_interface name="velocity" />
         </joint>
         <joint name="susRight_joint_b">
-            <command_interface name="velocity">
-                <param name="min">-1</param>
-                <param name="max">1</param>
-            </command_interface>
             <state_interface name="position" />
-            <state_interface name="velocity" />
         </joint>
         <joint name="wheel1_joint">

File: src/rover_description/urdf/rover_gazebo.xacro (robot description, xacro)
@@ -2,4 +2,13 @@
 <robot name="scarab"
   xmlns:xacro="http://ros.org/wiki/xacro">
+  <gazebo reference="wheel1_link">
+    <mu1>1000000000000000.0</mu1>
+    <mu2>1000000000000000.0</mu2>
+    <kp>1000000000000.0</kp>
+    <kd>10.0</kd>
+    <minDepth>0.001</minDepth>
+    <maxVel>0.1</maxVel>
+    <fdir1>1 0 0</fdir1>
+  </gazebo>
   <gazebo reference="wheel1_link">
     <mu1>1000000000000000.0</mu1>
