Commit message: Fix camera pointing backwards

File: src/rover_description/urdf/sensors/realsense.xacro (robot description, xacro)
@@ -5,5 +5,5 @@
     <parent link="body_link"/>
     <child link="realsense_link"/>
-    <origin xyz="-0.36 0.0 0.12" rpy="0.0 0.0 0.0"/>
+    <origin xyz="-0.36 0.0 0.12" rpy="0.0 0.0 ${pi}"/>
   </joint>
   <link name="realsense_link">

Commit message: Add realsense model

File: src/rover_description/urdf/sensors/realsense.xacro (robot description, xacro)
@@ -5,13 +5,13 @@
     <parent link="body_link"/>
     <child link="realsense_link"/>
-    <origin xyz="-0.36 0.0 0.12" rpy="0.0 0.0 ${pi}"/>
+    <origin xyz="-0.34 0.0 0.08" rpy="0.0 0.0 ${pi}"/>
   </joint>
   <link name="realsense_link">
     <visual>
       <geometry>
-        <box size="0.010 0.03 0.03"/>
+        <mesh filename="package://rover_description/meshes/d435.dae" scale="1 1 1"/>
       </geometry>
-      <material name="yellow">
-        <color rgba="1 1 0 1"/>
+      <material name="white">
+        <color rgba="0.9 0.9 0.9 1.0"/>
       </material>
     </visual>

Commit message: Feat: Add depth camera working with rtab

File: src/rover_description/urdf/sensors/realsense.xacro (robot description, xacro)
@@ -5,5 +5,5 @@
     <parent link="body_link"/>
     <child link="realsense_link"/>
-    <origin xyz="-0.34 0.0 0.08" rpy="0.0 0.0 ${pi}"/>
+    <origin xyz="-0.39 0.0 0.08" rpy="0.0 0.0 ${pi}"/>
   </joint>
   <link name="realsense_link">
@@ -32,7 +32,7 @@
         <horizontal_fov>1.085595</horizontal_fov>
         <image>
-          <width>1920</width>
-          <height>1080</height>
-          <format>RGB_INT8</format>
+          <width>640</width>
+          <height>480</height>
+          <format>R8G8B8</format>
         </image>
         <camera_info_topic>/camera/camera_info</camera_info_topic>
@@ -58,5 +58,5 @@
   </gazebo>
   <gazebo reference="realsense_link">
-    <sensor name="rgbd_camera" type="rgbd_camera">
+    <sensor name="rgbd_camera" type="depth_camera">
       <ignition_frame_id>realsense_link</ignition_frame_id>
       <camera name="rgbd_camera_frame">
@@ -80,7 +80,7 @@
         </distortion>
         <image>
-          <width>1280</width>
-          <height>720</height>
-          <format>L8</format>
+          <width>640</width>
+          <height>480</height>
+          <format>R8G8B8</format>
         </image>
         <clip>
@@ -93,4 +93,5 @@
             <far>10</far>
           </clip>
+          <output>depth</output>
         </depth_camera>
         <noise>
@@ -100,8 +101,8 @@
         </noise>
       </camera>
+      <topic>depth_camera</topic>
       <always_on>1</always_on>
       <update_rate>10</update_rate>
-      <visualize>0</visualize>
-      <topic>depth_camera</topic>
+      <visualize>1</visualize>
     </sensor>
   </gazebo>

Commit message: Feat: Get image and depth from gazebo rgbd_camera

File: src/rover_description/urdf/sensors/realsense.xacro (robot description, xacro)
@@ -17,4 +17,15 @@
     </visual>
   </link>
+  <joint name="imu_joint" type="fixed">
+    <parent link="realsense_link" />
+    <child link="imu_link"  />
+  </joint>
+  <link name="imu_link">
+    <visual>
+      <geometry>
+        <box size="0.1 0.1 0.1"/>
+      </geometry>
+    </visual>
+  </link>
   <!-- Optical joint will rotate the camera because it uses a different coordinate system where two axis are inverted -->
   <joint name="realsense_optical_joint" type="fixed">
@@ -32,7 +43,7 @@
         <horizontal_fov>1.085595</horizontal_fov>
         <image>
-          <width>640</width>
-          <height>480</height>
-          <format>R8G8B8</format>
+          <width>1920</width>
+          <height>1080</height>
+          <format>RGB_INT8</format>
         </image>
         <camera_info_topic>/camera/camera_info</camera_info_topic>
@@ -58,5 +69,5 @@
   </gazebo>
   <gazebo reference="realsense_link">
-    <sensor name="rgbd_camera" type="depth_camera">
+    <sensor name="rgbd_camera" type="rgbd_camera">
       <ignition_frame_id>realsense_link</ignition_frame_id>
       <camera name="rgbd_camera_frame">
@@ -80,7 +91,7 @@
         </distortion>
         <image>
-          <width>640</width>
-          <height>480</height>
-          <format>R8G8B8</format>
+          <width>1280</width>
+          <height>720</height>
+          <format>L8</format>
         </image>
         <clip>
@@ -93,5 +104,4 @@
             <far>10</far>
           </clip>
-          <output>depth</output>
         </depth_camera>
         <noise>
@@ -101,8 +111,21 @@
         </noise>
       </camera>
-      <topic>depth_camera</topic>
       <always_on>1</always_on>
       <update_rate>10</update_rate>
-      <visualize>1</visualize>
+      <visualize>0</visualize>
+      <topic>depth_camera</topic>
+    </sensor>
+  </gazebo>
+  <gazebo reference="imu_link">
+    <gravity>true</gravity>
+    <sensor name="imu_sensor" type="imu">
+      <ignition_frame_id>imu_link</ignition_frame_id>
+      <always_on>true</always_on>
+      <update_rate>25</update_rate>
+      <visualize>false</visualize>
+      <topic>imu</topic>
+      <plugin filename="libignition-gazebo-imu-system.so" name="ignition::gazebo::systems::Imu">
+      </plugin>
+      <pose>0 0 0 0 0 0</pose>
     </sensor>
   </gazebo>

Commit message: Feat: Add imu link to improve VO on RTAB

File: src/rover_description/urdf/sensors/realsense.xacro (robot description, xacro)
@@ -24,5 +24,5 @@
     <visual>
       <geometry>
-        <box size="0.1 0.1 0.1"/>
+        <box size="0.001 0.001 0.001"/>
       </geometry>
     </visual>
@@ -102,5 +102,5 @@
           <clip>
             <near>0.1</near>
-            <far>10</far>
+            <far>100</far>
           </clip>
         </depth_camera>
@@ -124,5 +124,5 @@
       <update_rate>25</update_rate>
       <visualize>false</visualize>
-      <topic>imu</topic>
+      <topic>imu/data_raw</topic>
       <plugin filename="libignition-gazebo-imu-system.so" name="ignition::gazebo::systems::Imu">
       </plugin>
