Commit message: Feat: Lint and format files

File: rover_description/urdf/sensors/realsense.xacro (robot description, xacro)
@@ -19,5 +19,5 @@
   <joint name="imu_joint" type="fixed">
     <parent link="realsense_link" />
-    <child link="imu_link"  />
+    <child link="imu_link" />
   </joint>
   <link name="imu_link">
