Commit message: feat: imporve sim speed disabling colissions on supension parts

File: rover_description/urdf/rover.urdf.xacro (robot description, xacro)
@@ -26,4 +26,5 @@
                 <!--<box size="1 0.6 0.3"/>-->
                 <mesh filename="package://rover_description/meshes/base_link.stl" scale="0.001 0.001 0.001" />
+                <!-- <box size="0.4 0.562228 0.12"/> -->
             </geometry>
             <material name="gray">
@@ -34,5 +35,6 @@
             <origin rpy="0 0 1.579795" xyz="0 0 0"/>
             <geometry>
-                <mesh filename="package://rover_description/meshes/base_link.stl" scale="0.001 0.001 0.001" />
+                <!-- <mesh filename="package://rover_description/meshes/base_link.stl" scale="0.001 0.001 0.001" /> -->
+                <box size="0.4 0.562228 0.12"/>
             </geometry>
         </collision>
@@ -60,10 +62,10 @@
             </material>
         </visual>
-        <collision>
+        <!-- <collision>
             <origin rpy="0 0 0" xyz="0 0 0"/>
             <geometry>
                 <mesh filename="package://rover_description/meshes/suspension_left_link_a.stl" scale="0.001 0.001 0.001" />
             </geometry>
-        </collision>
+        </collision> -->
     </link>
     <joint name="susLeft_joint_b" type="continuous">
@@ -90,10 +92,10 @@
             </material>
         </visual>
-        <collision>
+        <!-- <collision>
             <origin rpy="0 0 0" xyz="0 0 0"/>
             <geometry>
                 <mesh filename="package://rover_description/meshes/suspension_left_link_b.stl" scale="0.001 0.001 0.001" />
             </geometry>
-        </collision>
+        </collision> -->
     </link>
     <!-- This is the right suspension assembly -->
@@ -121,10 +123,10 @@
             </material>
         </visual>
-        <collision>
+        <!-- <collision>
             <origin rpy="0 0 0" xyz="0 0 0"/>
             <geometry>
                 <mesh filename="package://rover_description/meshes/suspension_right_link_a.stl" scale="0.001 0.001 0.001" />
             </geometry>
-        </collision>
+        </collision> -->
     </link>
     <joint name="susRight_joint_b" type="continuous">
@@ -149,10 +151,10 @@
             </material>
         </visual>
-        <collision>
+        <!-- <collision>
             <origin rpy="0 0 0" xyz="0 0 0"/>
             <geometry>
                 <mesh filename="package://rover_description/meshes/suspension_right_link_b.stl" scale="0.001 0.001 0.001" />
             </geometry>
-        </collision>
+        </collision> -->
     </link>
     <!-- This is the front right wheel of the rover -->
